Commit message: Update ROS 2 motion planning packages, clean track setup

File: src/medical_wheelchair/urdf/wheelchair.xacro (robot description, xacro)
@@ -261,3 +261,39 @@
     </plugin>
   </gazebo>
+  <!-- Lidar Sensor -->
+  <link name="laser_frame">
+    <xacro:cylinder_inertia m="0.2" r="0.05" h="0.05"/>
+    <visual>
+      <geometry><cylinder radius="0.05" length="0.05"/></geometry>
+      <material name="black"/>
+    </visual>
+  </link>
+  <joint name="laser_joint" type="fixed">
+    <parent link="base_link"/>
+    <child link="laser_frame"/>
+    <origin xyz="0.2 0 0.1" rpy="0 0 0"/>
+  </joint>
+  <gazebo reference="laser_frame">
+    <sensor name="gpu_lidar" type="gpu_lidar">
+      <topic>scan</topic>
+      <update_rate>10</update_rate>
+      <lidar>
+        <scan>
+          <horizontal>
+            <samples>360</samples>
+            <resolution>1</resolution>
+            <min_angle>-3.14159</min_angle>
+            <max_angle>3.14159</max_angle>
+          </horizontal>
+        </scan>
+        <range>
+          <min>0.08</min>
+          <max>10.0</max>
+          <resolution>0.01</resolution>
+        </range>
+      </lidar>
+      <always_on>1</always_on>
+      <visualize>true</visualize>
+    </sensor>
+  </gazebo>
 </robot>

Commit message: auto move

File: src/medical_wheelchair/urdf/wheelchair.xacro (robot description, xacro)
@@ -36,10 +36,6 @@
     </link>
   </xacro:macro>
-  <!-- Base Footprint -->
+  <!-- Base Footprint: No inertia for root link -->
   <link name="base_footprint">
-    <inertial>
-      <mass value="0.01"/>
-      <inertia ixx="0.0001" ixy="0" ixz="0" iyy="0.0001" iyz="0" izz="0.0001"/>
-    </inertial>
   </link>
   <joint name="base_footprint_joint" type="fixed">
@@ -168,6 +164,4 @@
       <child link="bogie_pivot_${side}"/>
       <origin xyz="0.15 0 0" rpy="0 0 0"/>
-      <axis xyz="0 1 0"/>
-      <limit effort="10" velocity="1" lower="-1.57" upper="1.57"/>
     </joint>
     <!-- Inverted V Bogie branches -->
@@ -289,5 +283,5 @@
         <range>
           <min>0.08</min>
-          <max>10.0</max>
+          <max>8.0</max>
           <resolution>0.01</resolution>
         </range>

Commit message: Add files via upload

File: src/medical_wheelchair/urdf/wheelchair.xacro (robot description, xacro)
@@ -196,9 +196,9 @@
       <collision>
         <origin xyz="0 0 0" rpy="1.5708 0 0"/>
-        <geometry><cylinder radius="0.07" length="0.05"/></geometry>
+        <geometry><sphere radius="0.07"/></geometry>
       </collision>
       <gazebo reference="front_${side}_wheel">
-        <mu1>0.1</mu1>
-        <mu2>0.1</mu2>
+        <mu1>0.001</mu1>
+        <mu2>0.001</mu2>
         <self_collide>false</self_collide>
       </gazebo>
@@ -221,9 +221,9 @@
       <collision>
         <origin xyz="0 0 0" rpy="1.5708 0 0"/>
-        <geometry><cylinder radius="0.07" length="0.05"/></geometry>
-      </collision>
-      <gazebo reference="front_${side}_wheel">
-        <mu1>0.1</mu1>
-        <mu2>0.1</mu2>
+        <geometry><sphere radius="0.07"/></geometry>
+      </collision>
+      <gazebo reference="middle_${side}_wheel">
+        <mu1>0.001</mu1>
+        <mu2>0.001</mu2>
         <self_collide>false</self_collide>
       </gazebo>
@@ -245,11 +245,16 @@
       name="gz::sim::systems::DiffDrive">
       <left_joint>rear_left_wheel_joint</left_joint>
-      <left_joint>middle_left_wheel_joint</left_joint>
-      <left_joint>front_left_wheel_joint</left_joint>
       <right_joint>rear_right_wheel_joint</right_joint>
-      <right_joint>middle_right_wheel_joint</right_joint>
-      <right_joint>front_right_wheel_joint</right_joint>
       <wheel_separation>0.35</wheel_separation>
       <wheel_radius>0.07</wheel_radius>
+      <odom_publish_frequency>50</odom_publish_frequency>
+      <max_linear_acceleration>2</max_linear_acceleration>
+      <min_linear_acceleration>-2</min_linear_acceleration>
+      <max_angular_acceleration>4</max_angular_acceleration>
+      <min_angular_acceleration>-4</min_angular_acceleration>
+      <max_linear_velocity>2</max_linear_velocity>
+      <min_linear_velocity>-2</min_linear_velocity>
+      <max_angular_velocity>4</max_angular_velocity>
+      <min_angular_velocity>-4</min_angular_velocity>
       <topic>/cmd_vel</topic>
     </plugin>

Commit message: Add files via upload

File: src/medical_wheelchair/urdf/wheelchair.xacro (robot description, xacro)
@@ -36,6 +36,10 @@
     </link>
   </xacro:macro>
-  <!-- Base Footprint: No inertia for root link -->
+  <!-- Base Footprint -->
   <link name="base_footprint">
+    <inertial>
+      <mass value="0.01"/>
+      <inertia ixx="0.0001" ixy="0" ixz="0" iyy="0.0001" iyz="0" izz="0.0001"/>
+    </inertial>
   </link>
   <joint name="base_footprint_joint" type="fixed">
@@ -46,5 +50,12 @@
   <!-- Base Link (Seat) -->
   <link name="base_link">
-    <xacro:box_inertia m="5.0" w="0.45" h="0.45" d="0.05"/>
+    <!-- Box Inertia expanded manually to adjust Center of Mass -->
+    <inertial>
+      <!-- Shift Center of Mass DOWN drastically to create a low gravity center -->
+      <origin xyz="0 0 -0.15" rpy="0 0 0"/>
+      <mass value="15.0"/>
+      <!-- Based on m=15.0, w=0.45, h=0.45, d=0.05 -->
+      <inertia ixx="0.25625" ixy="0" ixz="0" iyy="0.25625" iyz="0" izz="0.50625"/>
+    </inertial>
     <visual>
       <geometry><box size="0.45 0.45 0.05"/></geometry>
@@ -57,5 +68,5 @@
   <!-- Backrest -->
   <link name="backrest">
-    <xacro:box_inertia m="2.0" w="0.05" h="0.45" d="0.5"/>
+    <xacro:box_inertia m="0.5" w="0.05" h="0.45" d="0.5"/>
     <visual>
       <geometry><box size="0.05 0.45 0.5"/></geometry>
@@ -94,5 +105,5 @@
   <!-- Main Chassis Hub -->
   <link name="chassis_hub">
-    <xacro:box_inertia m="2.0" w="0.2" h="0.3" d="0.05"/>
+    <xacro:box_inertia m="10.0" w="0.2" h="0.3" d="0.05"/>
     <visual>
       <origin xyz="0 0 0" rpy="0 0 0"/>
@@ -110,172 +121,44 @@
     <origin xyz="0 0 -0.05" rpy="0 0 0"/>
   </joint>
-  <!-- Navigation Macros for Sides -->
-  <xacro:macro name="chassis_side" params="side reflect">
-    <!-- Rear Sloped Arm -->
-    <xacro:tubular_link name="rear_arm_${side}" length="0.25" radius="0.02" m="0.5" material="silver"/>
-    <joint name="rear_arm_${side}_joint" type="fixed">
-      <parent link="chassis_hub"/>
-      <child link="rear_arm_${side}"/>
-      <!--change-->
-      <origin xyz="-0.1 ${reflect * 0.15} 0" rpy="0 1.2 3.14159"/>
-    </joint>
-    <!-- Rear Wheel -->
-    <link name="rear_${side}_wheel">
-      <xacro:cylinder_inertia m="0.8" r="0.07" h="0.05"/>
-      <visual>
-        <origin xyz="0 0 0" rpy="1.5708 0 0"/>
-        <geometry><cylinder radius="0.07" length="0.05"/></geometry>
-        <material name="black"/>
-      </visual>
-      <collision>
-        <origin xyz="0 0 0" rpy="1.5708 0 0"/>
-        <geometry><cylinder radius="0.07" length="0.05"/></geometry>
-      </collision>
-      <gazebo reference="rear_${side}_wheel">
-        <mu1>1.0</mu1>
-        <mu2>1.0</mu2>
-        <self_collide>false</self_collide>
-      </gazebo>
-    </link>
-    <joint name="rear_${side}_wheel_joint" type="continuous">
-      <parent link="rear_arm_${side}"/>
-      <child link="rear_${side}_wheel"/>
-      <origin xyz="0.25 0 0" rpy="0 -1.2 0"/>
-      <axis xyz="0 1 0"/>
-    </joint>
-    <!-- Front Sloped Arm -->
-    <xacro:tubular_link name="front_arm_${side}" length="0.15" radius="0.02" m="0.3" material="silver"/>
-    <joint name="front_arm_${side}_joint" type="fixed">
-      <parent link="chassis_hub"/>
-      <child link="front_arm_${side}"/>
-      <origin xyz="0.1 ${reflect * 0.15} 0" rpy="0 0.8 0"/>
-    </joint>
-    <!-- Bogie Pivot -->
-    <link name="bogie_pivot_${side}">
-      <xacro:cylinder_inertia m="0.1" r="0.015" h="0.05"/>
-      <visual>
-        <origin xyz="0 0 0" rpy="1.5708 0 0"/>
-        <geometry><cylinder radius="0.015" length="0.05"/></geometry>
-        <material name="grey"/>
-      </visual>
-    </link>
-    <joint name="bogie_pivot_${side}_joint" type="fixed">
-      <parent link="front_arm_${side}"/>
-      <child link="bogie_pivot_${side}"/>
-      <origin xyz="0.15 0 0" rpy="0 0 0"/>
-    </joint>
-    <!-- Inverted V Bogie branches -->
-    <!-- Middle branch -->
-    <xacro:tubular_link name="bogie_middle_arm_${side}" length="0.15" radius="0.015" m="0.2" material="silver"/>
-    <joint name="bogie_middle_arm_joint_${side}" type="fixed">
-      <parent link="bogie_pivot_${side}"/>
-      <child link="bogie_middle_arm_${side}"/>
-      <!--change-->
-      <origin xyz="0 0 0" rpy="0 1.38 0"/>
-      <axis xyz="0 1 0"/>
-      <limit effort="10" velocity="1" lower="-3.14" upper="3.14"/>
-    </joint>
-    <!-- Front branch -->
-    <xacro:tubular_link name="bogie_front_arm_${side}" length="0.15" radius="0.015" m="0.2" material="silver"/>
-    <joint name="bogie_front_arm_joint_${side}" type="fixed">
-      <parent link="bogie_pivot_${side}"/>
-      <child link="bogie_front_arm_${side}"/>
-      <!--change-->
-      <origin xyz="0 0 0" rpy="0 0.16 0"/>
-      <axis xyz="0 1 0"/>
-      <limit effort="10" velocity="1" lower="-3.14" upper="3.14"/>
-    </joint>
-    <!-- Front Wheel -->
-    <link name="front_${side}_wheel">
-      <xacro:cylinder_inertia m="0.5" r="0.07" h="0.05"/>
-      <visual>
-        <origin xyz="0 0 0" rpy="1.5708 0 0"/>
-        <geometry><cylinder radius="0.07" length="0.05"/></geometry>
-        <material name="black"/>
-      </visual>
-      <collision>
-        <origin xyz="0 0 0" rpy="1.5708 0 0"/>
-        <geometry><sphere radius="0.07"/></geometry>
-      </collision>
-      <gazebo reference="front_${side}_wheel">
-        <mu1>0.001</mu1>
-        <mu2>0.001</mu2>
-        <self_collide>false</self_collide>
-      </gazebo>
-    </link>
-    <joint name="front_${side}_wheel_joint" type="continuous">
-      <parent link="bogie_front_arm_${side}"/>
-      <child link="front_${side}_wheel"/>
-      <!--change-->
-      <origin xyz="0.15 0 0" rpy="0 -0.16 0"/>
-      <axis xyz="0 1 0"/>
-    </joint>
-    <!-- Middle Wheel -->
-    <link name="middle_${side}_wheel">
-      <xacro:cylinder_inertia m="0.5" r="0.07" h="0.05"/>
-      <visual>
-        <origin xyz="0 0 0" rpy="1.5708 0 0"/>
-        <geometry><cylinder radius="0.07" length="0.05"/></geometry>
-        <material name="black"/>
-      </visual>
-      <collision>
-        <origin xyz="0 0 0" rpy="1.5708 0 0"/>
-        <geometry><sphere radius="0.07"/></geometry>
-      </collision>
-      <gazebo reference="middle_${side}_wheel">
-        <mu1>0.001</mu1>
-        <mu2>0.001</mu2>
-        <self_collide>false</self_collide>
-      </gazebo>
-    </link>
-    <joint name="middle_${side}_wheel_joint" type="continuous">
-      <parent link="bogie_middle_arm_${side}"/>
-      <child link="middle_${side}_wheel"/>
-      <!--change-->
-      <origin xyz="0.15 0 0" rpy="0 -1.38 0"/>
-      <axis xyz="0 1 0"/>
-    </joint>
-  </xacro:macro>
-  <xacro:chassis_side side="left" reflect="1"/>
-  <xacro:chassis_side side="right" reflect="-1"/>
-  <!-- Gazebo Plugins -->
-  <gazebo>
-    <plugin
-      filename="gz-sim-diff-drive-system"
-      name="gz::sim::systems::DiffDrive">
-      <left_joint>rear_left_wheel_joint</left_joint>
-      <right_joint>rear_right_wheel_joint</right_joint>
-      <wheel_separation>0.35</wheel_separation>
-      <wheel_radius>0.07</wheel_radius>
-      <odom_publish_frequency>50</odom_publish_frequency>
-      <max_linear_acceleration>2</max_linear_acceleration>
-      <min_linear_acceleration>-2</min_linear_acceleration>
-      <max_angular_acceleration>4</max_angular_acceleration>
-      <min_angular_acceleration>-4</min_angular_acceleration>
-      <max_linear_velocity>2</max_linear_velocity>
-      <min_linear_velocity>-2</min_linear_velocity>
-      <max_angular_velocity>4</max_angular_velocity>
-      <min_angular_velocity>-4</min_angular_velocity>
-      <topic>/cmd_vel</topic>
-    </plugin>
-  </gazebo>
-  <!-- Lidar Sensor -->
-  <link name="laser_frame">
-    <xacro:cylinder_inertia m="0.2" r="0.05" h="0.05"/>
-    <visual>
-      <geometry><cylinder radius="0.05" length="0.05"/></geometry>
-      <material name="black"/>
-    </visual>
-  </link>
-  <joint name="laser_joint" type="fixed">
-    <parent link="base_link"/>
-    <child link="laser_frame"/>
-    <origin xyz="0.2 0 0.1" rpy="0 0 0"/>
-  </joint>
-  <gazebo reference="laser_frame">
+  <!-- LiDAR Sensor & Mount -->
+  <link name="lidar_mount">
+    <visual>
+      <origin xyz="0 0 0" rpy="0 0 0"/>
+      <geometry><box size="0.05 0.05 0.1"/></geometry>
+      <material name="silver"/>
+    </visual>
+  </link>
+  <joint name="lidar_mount_joint" type="fixed">
+    <parent link="base_link"/>
+    <child link="lidar_mount"/>
+    <origin xyz="0.25 0 -0.05" rpy="0 0 0"/> <!-- At the front edge of the seat base, angled down -->
+  </joint>
+  <link name="lidar_link">
+    <inertial>
+      <mass value="0.1"/>
+      <inertia ixx="0.0001" ixy="0" ixz="0" iyy="0.0001" iyz="0" izz="0.0001"/>
+    </inertial>
+    <visual>
+      <origin xyz="0 0 0" rpy="0 0 0"/>
+      <geometry><cylinder radius="0.04" length="0.05"/></geometry>
+      <material name="fabric_red"/>
+    </visual>
+    <collision>
+      <origin xyz="0 0 0" rpy="0 0 0"/>
+      <geometry><cylinder radius="0.04" length="0.05"/></geometry>
+    </collision>
+  </link>
+  <joint name="lidar_joint" type="fixed">
+    <parent link="lidar_mount"/>
+    <child link="lidar_link"/>
+    <origin xyz="0.03 0 0.05" rpy="0 0 0"/>
+  </joint>
+  <gazebo reference="lidar_link">
     <sensor name="gpu_lidar" type="gpu_lidar">
-      <topic>scan</topic>
+      <pose>0 0 0 0 0 0</pose>
+      <topic>/scan</topic>
+      <ignition_frame_id>wheelchair/lidar_link</ignition_frame_id>
       <update_rate>10</update_rate>
-      <lidar>
+      <ray>
         <scan>
           <horizontal>
@@ -287,12 +170,174 @@
         </scan>
         <range>
-          <min>0.08</min>
-          <max>8.0</max>
+          <min>0.12</min>
+          <max>10.0</max>
           <resolution>0.01</resolution>
         </range>
-      </lidar>
-      <always_on>1</always_on>
+      </ray>
       <visualize>true</visualize>
     </sensor>
   </gazebo>
+  <!-- Navigation Macros for Sides -->
+  <xacro:macro name="chassis_side" params="side reflect">
+    <!-- Rear Sloped Arm -->
+    <xacro:tubular_link name="rear_arm_${side}" length="0.25" radius="0.02" m="0.5" material="silver"/>
+    <joint name="rear_arm_${side}_joint" type="fixed">
+      <parent link="chassis_hub"/>
+      <child link="rear_arm_${side}"/>
+      <origin xyz="-0.1 ${reflect * 0.15} 0" rpy="0 1.2 3.14159"/>
+    </joint>
+    <!-- Rear Wheel -->
+    <link name="rear_${side}_wheel">
+      <xacro:cylinder_inertia m="0.8" r="0.07" h="0.05"/>
+      <visual>
+        <origin xyz="0 0 0" rpy="1.5708 0 0"/>
+        <geometry><cylinder radius="0.07" length="0.05"/></geometry>
+        <material name="black"/>
+      </visual>
+      <collision>
+        <origin xyz="0 0 0" rpy="1.5708 0 0"/>
+        <geometry><sphere radius="0.07"/></geometry>
+      </collision>
+      <gazebo reference="rear_${side}_wheel">
+        <mu1>0.8</mu1>
+        <mu2>0.8</mu2>
+        <self_collide>false</self_collide>
+      </gazebo>
+    </link>
+    <joint name="rear_${side}_wheel_joint" type="continuous">
+      <parent link="rear_arm_${side}"/>
+      <child link="rear_${side}_wheel"/>
+      <origin xyz="0.25 0 0" rpy="0 -1.2 0"/>
+      <axis xyz="0 -1 0"/>
+      <limit effort="200" velocity="15"/>
+    </joint>
+    <!-- Front Sloped Arm -->
+    <xacro:tubular_link name="front_arm_${side}" length="0.15" radius="0.02" m="0.5" material="silver"/>
+    <joint name="front_arm_${side}_joint" type="fixed">
+      <parent link="chassis_hub"/>
+      <child link="front_arm_${side}"/>
+      <origin xyz="0.1 ${reflect * 0.15} 0" rpy="0 0.8 0"/>
+    </joint>
+    <!-- Bogie Pivot -->
+    <link name="bogie_pivot_${side}">
+      <xacro:cylinder_inertia m="0.1" r="0.015" h="0.05"/>
+      <visual>
+        <origin xyz="0 0 0" rpy="1.5708 0 0"/>
+        <geometry><cylinder radius="0.015" length="0.05"/></geometry>
+        <material name="grey"/>
+      </visual>
+    </link>
+    <joint name="bogie_pivot_${side}_joint" type="revolute">
+      <parent link="front_arm_${side}"/>
+      <child link="bogie_pivot_${side}"/>
+      <origin xyz="0.15 0 0" rpy="0 0 0"/>
+      <axis xyz="0 1 0"/>
+      <limit effort="10" velocity="1" lower="-0.5" upper="0.5"/>
+      <dynamics damping="1.0" friction="0.1"/>
+    </joint>
+    <!-- Inverted V Bogie branches -->
+    <!-- Middle branch -->
+    <xacro:tubular_link name="bogie_middle_arm_${side}" length="0.15" radius="0.015" m="0.3" material="silver"/>
+    <joint name="bogie_middle_arm_joint_${side}" type="fixed">
+      <parent link="bogie_pivot_${side}"/>
+      <child link="bogie_middle_arm_${side}"/>
+      <origin xyz="0 0 0" rpy="0 1.38 0"/>
+    </joint>
+    <!-- Front branch -->
+    <xacro:tubular_link name="bogie_front_arm_${side}" length="0.15" radius="0.015" m="0.3" material="silver"/>
+    <joint name="bogie_front_arm_joint_${side}" type="fixed">
+      <parent link="bogie_pivot_${side}"/>
+      <child link="bogie_front_arm_${side}"/>
+      <origin xyz="0 0 0" rpy="0 0.16 0"/>
+    </joint>
+    <!-- Front Wheel -->
+    <link name="front_${side}_wheel">
+      <xacro:cylinder_inertia m="0.5" r="0.07" h="0.05"/>
+      <visual>
+        <origin xyz="0 0 0" rpy="1.5708 0 0"/>
+        <geometry><cylinder radius="0.07" length="0.05"/></geometry>
+        <material name="black"/>
+      </visual>
+      <collision>
+        <origin xyz="0 0 0" rpy="1.5708 0 0"/>
+        <geometry><sphere radius="0.07"/></geometry>
+      </collision>
+      <gazebo reference="front_${side}_wheel">
+        <mu1>0.8</mu1>
+        <mu2>0.8</mu2>
+        <self_collide>false</self_collide>
+      </gazebo>
+    </link>
+    <joint name="front_${side}_wheel_joint" type="continuous">
+      <parent link="bogie_front_arm_${side}"/>
+      <child link="front_${side}_wheel"/>
+      <origin xyz="0.15 0 0" rpy="0 -0.16 0"/>
+      <axis xyz="0 1 0"/>
+      <limit effort="200" velocity="15"/>
+    </joint>
+    <!-- Middle Wheel -->
+    <link name="middle_${side}_wheel">
+      <xacro:cylinder_inertia m="0.5" r="0.07" h="0.05"/>
+      <visual>
+        <origin xyz="0 0 0" rpy="1.5708 0 0"/>
+        <geometry><cylinder radius="0.07" length="0.05"/></geometry>
+        <material name="black"/>
+      </visual>
+      <collision>
+        <origin xyz="0 0 0" rpy="1.5708 0 0"/>
+        <geometry><sphere radius="0.07"/></geometry>
+      </collision>
+      <gazebo reference="middle_${side}_wheel">
+        <mu1>0.8</mu1>
+        <mu2>0.8</mu2>
+        <self_collide>false</self_collide>
+      </gazebo>
+    </link>
+    <joint name="middle_${side}_wheel_joint" type="continuous">
+      <parent link="bogie_middle_arm_${side}"/>
+      <child link="middle_${side}_wheel"/>
+      <origin xyz="0.15 0 0" rpy="0 -1.38 0"/>
+      <axis xyz="0 1 0"/>
+      <limit effort="200" velocity="15"/>
+    </joint>
+  </xacro:macro>
+  <xacro:chassis_side side="left" reflect="1"/>
+  <xacro:chassis_side side="right" reflect="-1"/>
+  <!-- Gazebo Plugins -->
+  <gazebo>
+    <plugin
+      filename="gz-sim-diff-drive-system"
+      name="gz::sim::systems::DiffDrive">
+      <namespace>/</namespace>
+      <left_joint>rear_left_wheel_joint</left_joint>
+      <left_joint>middle_left_wheel_joint</left_joint>
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